File: Abschluss/Abschluss/Abschluss.sch (KiCad schematic (older format))
At the start: 26 parts, among them J1 Conn_01x04, J2 Photo, J3 Photo, J4 Motor, J5 Bat, J6 Erweiterung, Q1 SFH309, SW1 Reset, U1 ESP-12F, U2 DS1307Z+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

Commit message: Rechtschreibprüfung
Other:
- note added: "2"
- note added: "20.01.2019"
- note added: "Hühnerklappe \n"
- moved on the sheet: BT1, J1, J2, J3, J4, J6, JP1, Q1, QZ1, R1, R2, R3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
